File: KiCAD/Pancake/DAC_Filters.sch (KiCad schematic (older format))
At the start: 23 parts

Commit message: Extra kicad stuff
Parts:
- removed R? (x4): R, symbol Device:R
- C? (x4): value C -> 680pF
- C? (x2): value C -> 220pF
- C? (x2): value C -> 2.2nF
- C? (x2): value C -> 150pF
- R? (x2): value R -> 31.6k
- R? (x2): value R -> 22.1k
- R? (x2): value R -> 10.7k
- R? (x2): value R -> 34.8k
Connections:
- net IN1: now also C?.2, R?.1
- net IN2: now also C?.2, R?.1
- net -12V: now reaches IC?.11 (VCC-)
- net +12V: now reaches IC?.4 (VCC+)
Other:
- note added: "1st pole"
- note removed: "1st pole and voltage divider"
- moved on the sheet: C?
