File: KiCAD/Pancake/Relays.sch (KiCad schematic (older format))
At the start: 29 parts

Commit message: Schematic almost complete. layout still required
Parts:
- gave numbers to parts that had none: 29
