File: KiCAD/Pancake/Relay.sch (KiCad schematic (older format))
At the start: 18 parts, among them Q901 ULN2003AIN, Q902 ULN2003AIN

Commit message: Models
Parts:
- Q901, Q902: symbol SamacSys_Parts:ULN2003AIN -> Pancake-rescue:ULN2003AIN-SamacSys_Parts
Changed lines of the file:
@@
 $EndComp
 $Comp
-L SamacSys_Parts:ULN2003AIN Q901
+L Pancake-rescue:ULN2003AIN-SamacSys_Parts Q901
 U 1 1 614225A7
 P 1250 2000
@@
 $EndComp
 $Comp
-L SamacSys_Parts:ULN2003AIN Q902
+L Pancake-rescue:ULN2003AIN-SamacSys_Parts Q902
 U 1 1 6149A825
 P 6200 1950

Commit message: Lib updates and capacitor add. Simulation on power resistor working
Parts:
- Q901: footprint DIP794W53P254L1930H508Q16N -> SamacSys_Parts:DIP794W53P254L1930H508Q16N; symbol Pancake-rescue:ULN2003AIN-SamacSys_Parts -> SamacSys_Parts:ULN2003AIN
- Q902: footprint DIP794W53P254L1930H508Q16N -> SamacSys_Parts:DIP794W53P254L1930H508Q16N
- RelayA901, RelayB901, RelayC901, RelayD901, RelayE901, RelayF901, RelayG901, RelayH901, RelayI901, RelayJ901: footprint 833H1AFS12VDC -> SamacSys_Parts:833H1AFS12VDC
Changed lines of the file:
@@
 F 0 "RelayA901" H 10500 1300 50  0000 C CNN
 F 1 "833H-1A-F-S-12VDC" H 10475 1076 50  0000 C CNN
-F 2 "833H1AFS12VDC" H 11050 1450 50  0001 L CNN
+F 2 "SamacSys_Parts:833H1AFS12VDC" H 11050 1450 50  0001 L CNN
 F 3 "https://eu.mouser.com/datasheet/2/378/20119191320287145-4912.pdf" H 10100 1750 50  0001 L CNN
 	1    9750 1350
@@
 F 0 "RelayD901" H 10400 3900 50  0000 C CNN
 F 1 "833H-1A-F-S-12VDC" H 10475 3626 50  0000 C CNN
-F 2 "833H1AFS12VDC" H 11050 4000 50  0001 L CNN
+F 2 "SamacSys_Parts:833H1AFS12VDC" H 11050 4000 50  0001 L CNN
 F 3 "https://eu.mouser.com/datasheet/2/378/20119191320287145-4912.pdf" H 10100 4300 50  0001 L CNN
 	1    9750 3900
@@
 F 0 "RelayB901" H 10425 2600 50  0000 C CNN
 F 1 "833H-1A-F-S-12VDC" H 10475 2326 50  0000 C CNN
-F 2 "833H1AFS12VDC" H 11050 2700 50  0001 L CNN
+F 2 "SamacSys_Parts:833H1AFS12VDC" H 11050 2700 50  0001 L CNN
 F 3 "https://eu.mouser.com/datasheet/2/378/20119191320287145-4912.pdf" H 10100 3000 50  0001 L CNN
 	1    9750 2600
@@
 F 0 "RelayC901" H 10425 3275 50  0000 C CNN
 F 1 "833H-1A-F-S-12VDC" H 10475 2976 50  0000 C CNN
-F 2 "833H1AFS12VDC" H 11050 3350 50  0001 L CNN
+F 2 "SamacSys_Parts:833H1AFS12VDC" H 11050 3350 50  0001 L CNN
 F 3 "https://eu.mouser.com/datasheet/2/378/20119191320287145-4912.pdf" H 10100 3650 50  0001 L CNN
 	1    9750 3250
@@
 F 0 "RelayG901" H 5450 2150 50  0000 C CNN
 F 1 "833H-1A-F-S-12VDC" H 5425 1926 50  0000 C CNN
-F 2 "833H1AFS12VDC" H 6000 2300 50  0001 L CNN
+F 2 "SamacSys_Parts:833H1AFS12VDC" H 6000 2300 50  0001 L CNN
 F 3 "https://eu.mouser.com/datasheet/2/378/20119191320287145-4912.pdf" H 5050 2600 50  0001 L CNN
 	1    4700 2200
@@
 F 0 "RelayF901" H 5450 1650 50  0000 C CNN
 F 1 "833H-1A-F-S-12VDC" H 5425 1426 50  0000 C CNN
-F 2 "833H1AFS12VDC" H 6000 1800 50  0001 L CNN
+F 2 "SamacSys_Parts:833H1AFS12VDC" H 6000 1800 50  0001 L CNN
 F 3 "https://eu.mouser.com/datasheet/2/378/20119191320287145-4912.pdf" H 5050 2100 50  0001 L CNN
 	1    4700 1700
@@
 F 0 "RelayE901" H 5450 1100 50  0000 C CNN
 F 1 "833H-1A-F-S-12VDC" H 5425 876 50  0000 C CNN
-F 2 "833H1AFS12VDC" H 6000 1250 50  0001 L CNN
+F 2 "SamacSys_Parts:833H1AFS12VDC" H 6000 1250 50  0001 L CNN
 F 3 "https://eu.mouser.com/datasheet/2/378/20119191320287145-4912.pdf" H 5050 1550 50  0001 L CNN
 	1    4700 1150
@@
 F 0 "RelayJ901" H 5400 4300 50  0000 C CNN
 F 1 "833H-1A-F-S-12VDC" H 5375 4076 50  0000 C CNN
-F 2 "833H1AFS12VDC" H 5950 4450 50  0001 L CNN
+F 2 "SamacSys_Parts:833H1AFS12VDC" H 5950 4450 50  0001 L CNN
 F 3 "https://eu.mouser.com/datasheet/2/378/20119191320287145-4912.pdf" H 5000 4750 50  0001 L CNN
 	1    4650 4350
@@
 F 0 "RelayI901" H 5400 3700 50  0000 C CNN
 F 1 "833H-1A-F-S-12VDC" H 5375 3526 50  0000 C CNN
-F 2 "833H1AFS12VDC" H 5950 3900 50  0001 L CNN
+F 2 "SamacSys_Parts:833H1AFS12VDC" H 5950 3900 50  0001 L CNN
 F 3 "https://eu.mouser.com/datasheet/2/378/20119191320287145-4912.pdf" H 5000 4200 50  0001 L CNN
 	1    4650 3800
@@
 F 0 "RelayH901" H 5400 3250 50  0000 C CNN
 F 1 "833H-1A-F-S-12VDC" H 5375 3026 50  0000 C CNN
-F 2 "833H1AFS12VDC" H 5950 3400 50  0001 L CNN
+F 2 "SamacSys_Parts:833H1AFS12VDC" H 5950 3400 50  0001 L CNN
 F 3 "https://eu.mouser.com/datasheet/2/378/20119191320287145-4912.pdf" H 5000 3700 50  0001 L CNN
 	1    4650 3300
@@
 $EndComp
 $Comp
-L Pancake-rescue:ULN2003AIN-SamacSys_Parts Q901
+L SamacSys_Parts:ULN2003AIN Q901
 U 1 1 614225A7
 P 1250 2000
 F 0 "Q901" H 1750 2265 50  0000 C CNN
 F 1 "ULN2003AIN" H 1750 2174 50  0000 C CNN
-F 2 "DIP794W53P254L1930H508Q16N" H 2100 2100 50  0001 L CNN
+F 2 "SamacSys_Parts:DIP794W53P254L1930H508Q16N" H 2100 2100 50  0001 L CNN
 F 3 "http://uk.rs-online.com/web/p/products/7320887" H 2100 2000 50  0001 L CNN
 F 4 "Texas Instruments ULN2003AINE4, 7-element NPN Darlington Pair, 500 mA 50 V, 16-Pin PDIP" H 2100 1900 50  0001 L CNN "Description"
@@
 F 0 "Q902" H 6700 2215 50  0000 C CNN
 F 1 "ULN2003AIN" H 6700 2124 50  0000 C CNN
-F 2 "DIP794W53P254L1930H508Q16N" H 7050 2050 50  0001 L CNN
+F 2 "SamacSys_Parts:DIP794W53P254L1930H508Q16N" H 7050 2050 50  0001 L CNN
 F 3 "http://uk.rs-online.com/web/p/products/7320887" H 7050 1950 50  0001 L CNN
 F 4 "Texas Instruments ULN2003AINE4, 7-element NPN Darlington Pair, 500 mA 50 V, 16-Pin PDIP" H 7050 1850 50  0001 L CNN "Description"
